File: team_test/team_test.kicad_sch (KiCad schematic)
At the start: 0 parts

Commit message: add mcu
Parts:
- added U1: STM32WB5MMG, RF_Module:ST-SiP-LGA-86-11x7.3mm, symbol RF_Module:STM32WB5MMG
Connections:
- new net: U1.31 (VSS), U1.5 (VSS), U1.57 (VSS), U1.60 (VSS), U1.84 (VSS), U1.86 (VSS)
Changed lines of the file:
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@@
 	(generator_version "9.0")
 	(paper "A4")
+	(symbol
+		(lib_id "RF_Module:STM32WB5MMG")
+		(at 139.7 92.71 0)
+		(unit 1)
+		(exclude_from_sim no)
+		(in_bom yes)
+		(on_board yes)
+		(dnp no)
+		(fields_autoplaced yes)
+		(property "Reference" "U1"
+			(at 144.3833 153.67 0)
+			(effects
+				(font
+					(size 1.27 1.27)
+				)
+				(justify left)
+			)
+		)
+		(property "Value" "STM32WB5MMG"
+			(at 144.3833 156.21 0)
+			(effects
+				(font
+					(size 1.27 1.27)
+				)
+				(justify left)
+			)
+		)
+		(property "Footprint" "RF_Module:ST-SiP-LGA-86-11x7.3mm"
+			(at 139.7 95.25 0)
+			(effects
+				(font
+					(size 1.27 1.27)
+				)
+				(hide yes)
+			)
+		)
+		(property "Datasheet" "https://www.st.com/resource/en/datasheet/stm32wb5mmg.pdf"
+			(at 139.7 92.71 0)
+			(effects
+				(font
+					(size 1.27 1.27)
+				)
+				(hide yes)
+			)
+		)
+		(property "Description" "ST Microelectronics STM32WB55VG ARM Cortex Bluetooth Low Energy 5.0, Zigbee and 802.15.4 module, 1 MB Flash, 256kb RAM, Fully integrated BOM"
+			(at 139.7 92.71 0)
+			(effects
+				(font
+					(size 1.27 1.27)
+				)
+				(hide yes)
+			)
+		)
+		(pin "77"
+		)
+		(pin "68"
+		)
+		(pin "78"
+		)
+		(pin "13"
+		)
+		(pin "80"
+		)
+		(pin "34"
+		)
+		(pin "81"
+		)
+		(pin "8"
+		)
+		(pin "67"
+		)
+		(pin "66"
+		)
+		(pin "64"
+		)
+		(pin "79"
+		)
+		(pin "24"
+		)
+		(pin "74"
+		)
+		(pin "61"
+		)
+		(pin "70"
+		)
+		(pin "72"
+		)
+		(pin "75"
+		)
+		(pin "82"
+		)
+		(pin "42"
+		)
+		(pin "33"
+		)
+		(pin "62"
+		)
+		(pin "65"
+		)
+		(pin "63"
+		)
+		(pin "73"
+		)
+		(pin "76"
+		)
+		(pin "12"
+		)
+		(pin "9"
+		)
+		(pin "7"
+		)
+		(pin "49"
+		)
+		(pin "36"
+		)
+		(pin "45"
+		)
+		(pin "71"
+		)
+		(pin "83"
+		)
+		(pin "69"
+		)
+		(pin "22"
+		)
+		(pin "23"
+		)
+		(pin "17"
+		)
+		(pin "31"
+		)
+		(pin "1"
+		)
+		(pin "53"
+		)
+		(pin "50"
+		)
+		(pin "85"
+		)
+		(pin "2"
+		)
+		(pin "3"
+		)
+		(pin "32"
+		)
+		(pin "56"
+		)
+		(pin "51"
+		)
+		(pin "15"
+		)
+		(pin "4"
+		)
+		(pin "57"
+		)
+		(pin "86"
+		)
+		(pin "28"
+		)
+		(pin "52"
+		)
+		(pin "16"
+		)
+		(pin "84"
+		)
+		(pin "60"
+		)
+		(pin "30"
+		)
+		(pin "29"
+		)
+		(pin "40"
+		)
+		(pin "6"
+		)
+		(pin "5"
+		)
+		(pin "55"
+		)
+		(pin "54"
+		)
+		(pin "21"
+		)
+		(pin "59"
+		)
+		(pin "35"
+		)
+		(pin "26"
+		)
+		(pin "46"
+		)
+		(pin "20"
+		)
+		(pin "14"
+		)
+		(pin "27"
+		)
+		(pin "18"
+		)
+		(pin "41"
+		)
+		(pin "25"
+		)
+		(pin "44"
+		)
+		(pin "11"
+		)
+		(pin "19"
+		)
+		(pin "37"
+		)
+		(pin "47"
+		)
+		(pin "48"
+		)
+		(pin "38"
+		)
+		(pin "58"
+		)
+		(pin "43"
+		)
+		(pin "39"
+		)
+		(pin "10"
+		)
+		(instances
+			(project ""
+				(path "/ae9df8f7-f70f-416f-9081-a067ae98461e"
+					(reference "U1")
+					(unit 1)
+				)
+			)
+		)
+	)
 	(sheet_instances
 		(path "/"

Commit message: second commit
Parts:
- added U3: AD8212, Package_SO:MSOP-8_3x3mm_P0.65mm, symbol Amplifier_Current:AD8212
- added U4: INA139, Package_TO_SOT_SMD:SOT-23-5, symbol Amplifier_Current:INA139
Changed lines of the file:
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@@
 	(paper "A4")
+	(symbol
+		(lib_id "Amplifier_Current:INA139")
+		(at 134.62 181.61 0)
+		(unit 1)
+		(exclude_from_sim no)
+		(in_bom yes)
+		(on_board yes)
+		(dnp no)
+		(fields_autoplaced yes)
+		(property "Reference" "U4"
+			(at 144.78 175.1898 0)
+			(effects
+				(font
+					(size 1.27 1.27)
+				)
+			)
+		)
+		(property "Value" "INA139"
+			(at 144.78 177.7298 0)
+			(effects
+				(font
+					(size 1.27 1.27)
+				)
+			)
+		)
+		(property "Footprint" "Package_TO_SOT_SMD:SOT-23-5"
+			(at 134.62 181.61 0)
+			(effects
+				(font
+					(size 1.27 1.27)
+				)
+				(hide yes)
+			)
+		)
+		(property "Datasheet" "http://www.ti.com/lit/ds/symlink/ina169.pdf"
+			(at 134.62 181.483 0)
+			(effects
+				(font
+					(size 1.27 1.27)
+				)
+				(hide yes)
+			)
+		)
+		(property "Description" "High-Side Measurement Current Shunt Monitor, 40V, SOT-23-5"
+			(at 134.62 181.61 0)
+			(effects
+				(font
+					(size 1.27 1.27)
+				)
+				(hide yes)
+			)
+		)
+		(pin "1"
+		)
+		(pin "3"
+		)
+		(pin "4"
+		)
+		(pin "5"
+		)
+		(pin "2"
+		)
+		(instances
+			(project ""
+				(path "/ae9df8f7-f70f-416f-9081-a067ae98461e"
+					(reference "U4")
+					(unit 1)
+				)
+			)
+		)
+	)
+	(symbol
+		(lib_id "Amplifier_Current:AD8212")
+		(at 41.91 148.59 0)
+		(unit 1)
+		(exclude_from_sim no)
+		(in_bom yes)
+		(on_board yes)
+		(dnp no)
+		(fields_autoplaced yes)
+		(property "Reference" "U3"
+			(at 41.91 158.75 0)
+			(effects
+				(font
+					(size 1.27 1.27)
+				)
+			)
+		)
+		(property "Value" "AD8212"
+			(at 41.91 161.29 0)
+			(effects
+				(font
+					(size 1.27 1.27)
+				)
+			)
+		)
+		(property "Footprint" "Package_SO:MSOP-8_3x3mm_P0.65mm"
+			(at 41.91 148.59 0)
+			(effects
+				(font
+					(size 1.27 1.27)
+				)
+				(justify left)
+				(hide yes)
+			)
+		)
+		(property "Datasheet" "https://www.analog.com/media/en/technical-documentation/data-sheets/AD8212.pdf"
+			(at 58.42 166.37 0)
+			(effects
+				(font
+					(size 1.27 1.27)
+				)
+				(hide yes)
+			)
+		)
+		(property "Description" "65V High Voltage Current, Shunt Monitor, adjustable gain, bandwidth 1000kHz, Vcc=7V~65V, current output, unidirectional, MSOP-8"
+			(at 41.91 148.59 0)
+			(effects
+				(font
+					(size 1.27 1.27)
+				)
+				(hide yes)
+			)
+		)
+		(pin "1"
+		)
+		(pin "8"
+		)
+		(pin "3"
+		)
+		(pin "7"
+		)
+		(pin "6"
+		)
+		(pin "5"
+		)
+		(pin "2"
+		)
+		(pin "4"
+		)
+		(instances
+			(project ""
+				(path "/ae9df8f7-f70f-416f-9081-a067ae98461e"
+					(reference "U3")
+					(unit 1)
+				)
+			)
+		)
+	)
 	(symbol
 		(lib_id "RF_Module:STM32WB5MMG")
