File: team_test/team_test.kicad_pcb (KiCad board)
At the start: 2 copper layers, 1 part, among them U1 STM32WB5MMG

Commit message: PCB update
Parts:
- added U3: AD8212, Package_SO:MSOP-8_3x3mm_P0.65mm, F.Cu at (132.0, 89.9)
- added U4: INA139, Package_TO_SOT_SMD:SOT-23-5, F.Cu at (159.6, 97.0)
